Commit message: Fix front_looking_sonar indentation in sonar_snippets.xacro

File: uuv_sensor_plugins/uuv_sensor_ros_plugins/urdf/sonar_snippets.xacro (robot description, xacro)
@@ -153,6 +153,6 @@
   </xacro:macro>
   <xacro:macro name="forward_looking_sonar"
-    params="namespace suffix parent_link topic mass update_rate
-      samples fov width height *inertia *origin">
+               params="namespace suffix parent_link topic mass update_rate
+                       samples fov width height *inertia *origin">
     <!-- Sensor link -->
     <link name="${namespace}/forward_sonar${suffix}_link">
@@ -179,8 +179,8 @@
       <sensor name="${namespace}/image_sonar" type="depth">
         <camera>
-		  <horizontal_fov>${fov}</horizontal_fov>
+	  <horizontal_fov>${fov}</horizontal_fov>
           <image>
-		    <width>${width}</width>
-		    <height>${height}</height>
+	    <width>${width}</width>
+	    <height>${height}</height>
             <format>R8G8B8</format>
           </image>
@@ -193,18 +193,18 @@
           </save>
         </camera>
-	    <plugin filename="libimage_sonar_ros_plugin.so" name="forward_sonar${suffix}_controller">
-		  <topicName>${topic}</topicName>
+	<plugin filename="libimage_sonar_ros_plugin.so" name="forward_sonar${suffix}_controller">
+	  <topicName>${topic}</topicName>
           <frameName>forward_sonar${suffix}_optical_frame</frameName>
         </plugin>
         <always_on>true</always_on>
-	    <update_rate>${update_rate}</update_rate>
+	<update_rate>${update_rate}</update_rate>
       </sensor>
     </gazebo>
-	<joint name="${namespace}/forward_sonar${suffix}_joint" type="fixed">
+    <joint name="${namespace}/forward_sonar${suffix}_joint" type="fixed">
       <origin xyz="0 0 0" rpy="${-pi/2} 0 ${-pi/2}"/>
       <parent link="${namespace}/forward_sonar${suffix}_link"/>
       <child link="${namespace}/forward_sonar${suffix}_optical_frame"/>
     </joint>
-	<link name="${namespace}/forward_sonar${suffix}_optical_frame"/>
+    <link name="${namespace}/forward_sonar${suffix}_optical_frame"/>
   </xacro:macro>
 </robot>
