Commit message: Add second, horizontally mounted sonar to sonar configuration

File: uuv_descriptions/robots/rexrov_sonar_cerqueira.xacro (robot description, xacro)
@@ -21,16 +21,28 @@
   <xacro:forward_looking_sonar
       namespace="${namespace}"
-      suffix="down"
+      suffix="horiz"
       parent_link="${namespace}/base_link"
-      topic="forward_sonar"
       mass="0.015"
       update_rate="40"
       samples="100"
-        fov="1.54719755"
-        width="768"
-        height="492">
-      <inertia ixx="0.00001" ixy="0.0" ixz="0.0" iyy="0.00001" iyz="0.0" izz="0.00001" />
-      <origin xyz="1.15 0 0.4" rpy="0 0.3 0"/>
-    </xacro:forward_looking_sonar>
+      fov="1.54719755"
+      width="768"
+      height="492">
+    <inertia ixx="0.00001" ixy="0.0" ixz="0.0" iyy="0.00001" iyz="0.0" izz="0.00001" />
+    <origin xyz="1.15 0 0.4" rpy="0 0.3 0"/>
+  </xacro:forward_looking_sonar>
+  <xacro:forward_looking_sonar
+      namespace="${namespace}"
+      suffix="vert"
+      parent_link="${namespace}/base_link"
+      mass="0.015"
+      update_rate="40"
+      samples="100"
+      fov="1.54719755"
+      width="768"
+      height="492">
+    <inertia ixx="0.00001" ixy="0.0" ixz="0.0" iyy="0.00001" iyz="0.0" izz="0.00001" />
+    <origin xyz="1.15 0 0.45" rpy="1.5707 0.3 0"/>
+  </xacro:forward_looking_sonar>
   <!-- Create the RexROV vehicle -->
   <xacro:rexrov_base
